File: Datalore-IP-m4-rev02.brd (EAGLE design)
At the start: 25.4 x 25.4 mm, 20 parts

Commit message: stated mother board
Routing:
- net GND: track 41.3 -> 45.9 mm
Changed lines of the file:
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@@
 <via x="5" y="9" extent="1-16" drill="0.2" diameter="0.125"/>
 <via x="8.5" y="25.25" extent="1-16" drill="0.2" diameter="0.125"/>
-<via x="6.75" y="25.25" extent="1-16" drill="0.2" diameter="0.125"/>
 <via x="12.25" y="19.25" extent="1-16" drill="0.2" diameter="0.125"/>
 <via x="10.5" y="21.75" extent="1-16" drill="0.2" diameter="0.125"/>
@@
 <wire x1="5.5" y1="15.75" x2="5.75" y2="15.75" width="0.3" layer="1"/>
 <contactref element="C1" pad="1"/>
-<wire x1="6.75" y1="25.25" x2="6.746" y2="25.254" width="0.3" layer="16"/>
-<wire x1="6.65246875" y1="25.254" x2="6.746" y2="25.254" width="0.3" layer="16"/>
-<wire x1="6.35" y1="25.55646875" x2="6.65246875" y2="25.254" width="0.3" layer="16"/>
-<wire x1="6.35" y1="25.65" x2="6.75" y2="25.25" width="0.3" layer="1"/>
 <wire x1="12.25" y1="19.25" x2="18.375" y2="13.125" width="0.3" layer="1"/>
 <wire x1="19" y1="18.75" x2="18.625" y2="18.375" width="0.3" layer="1"/>
 <wire x1="18.625" y1="18.375" x2="18.375" y2="18.375" width="0.3" layer="1"/>
-<wire x1="18.375" y1="18.375" x2="13.25" y2="13.25" width="0.3" layer="1"/>
 <via x="13" y="5.375" extent="1-16" drill="0.2" diameter="0.125"/>
-<wire x1="6.35" y1="26.67" x2="6.35" y2="25.65" width="0.2" layer="1"/>
-<wire x1="6.35" y1="26.67" x2="6.35" y2="25.65" width="0.2" layer="16"/>
-<wire x1="6.35" y1="25.65" x2="6.75" y2="25.25" width="0.2" layer="16"/>
 <via x="2.75" y="25.25" extent="1-16" drill="0.2" diameter="0.125"/>
+<wire x1="19" y1="18.75" x2="14" y2="13.75" width="0.2" layer="1"/>
+<wire x1="14" y1="13.75" x2="13.75" y2="13.75" width="0.2" layer="1"/>
+<wire x1="15.75" y1="15.75" x2="12.25" y2="12.25" width="0.2" layer="1"/>
+<wire x1="6.35" y1="26.67" x2="6.35" y2="25.4" width="0.3" layer="16"/>
+<wire x1="6.35" y1="25.4" x2="6.625" y2="25.125" width="0.3" layer="16"/>
+<via x="6.625" y="25.125" extent="1-16" drill="0.2" diameter="0.125"/>
+<wire x1="6.35" y1="26.67" x2="6.35" y2="25.4" width="0.3" layer="1"/>
+<wire x1="6.35" y1="25.4" x2="6.625" y2="25.125" width="0.3" layer="1"/>
 </signal>
 <signal name="FLASH_IO2">
